File: KiCad/latte.kicad_pcb (KiCad board)
At the start: 2 copper layers, 347.8 x 94.7 mm, 151 parts, among them J1 Conn_01x04, U1 ATmega32U4-AU, Y1 Resonator_Small

Commit message: placed components
Parts:
- removed the 1.5u6 at (-12.0, -39.7)
- removed 1.5u7, 1.5u8: MX-NoLED, MX_Only:MXOnly-1.5U-NoLED
- added 1.5u5: MX-NoLED, MX_Only:MXOnly-1.5U-NoLED, F.Cu at (208.5, 166.6)
- added D66: D_Small, Footprints:D_SOD-123-Pretty, F.Cu at (0.69, -15.7)
- added MX57: MX-NoLED, MX_Only:MXOnly-1U-NoLED, F.Cu at (280.0, 139.2)
- added MX58: MX-NoLED, MX_Only:MXOnly-1U-NoLED, F.Cu at (299.1, 139.2)
- added MX59: MX-NoLED, MX_Only:MXOnly-1U-NoLED, F.Cu at (318.1, 139.2)
- added R2: 220, Footprints:R_0805_2012Metric, F.Cu at (95.5, 19.0)
- 10u1: footprint Footprints:MX-10U -> Footprints:MXOnly-10U-NoLED
- moved 10u1 370.0 mm to (114.3, 193.9)
- moved 1.5u6 289.1 mm to (251.4, 139.2)
- moved 1.5u4 220.8 mm to (13.3, 139.2)
- renumbered 1.5u5 to 1.5u6, D66 to D67, D67 to D68, D68 to D69, D69 to D70, R2 to R3, R3 to R4, R4 to R5
Connections:
- MX1 pad 1: unconnected-(MX1-Pad1) -> COL0

Commit message: honestly bro i forget what i did here
Parts:
- added C2: 10uF, keeb:C_0805_2012Metric, B.Cu at (274.1, 91.7)
- added C3: .1uF, keeb:C_0805_2012Metric, B.Cu at (284.7, 102.2)
- added C4: .1uF, keeb:C_0805_2012Metric, B.Cu at (274.1, 112.8)
- added C5: .1uF, keeb:C_0805_2012Metric, B.Cu at (263.6, 102.2)
- added C6: 22pF, keeb:C_0805_2012Metric, B.Cu at (279.7, 90.8)
- added C7: 22pF, keeb:C_0805_2012Metric, B.Cu at (285.2, 96.2)
- added C8: .1uF, keeb:C_0805_2012Metric, B.Cu at (267.6, 93.3)
- 10u1: footprint Footprints:MXOnly-10U-NoLED -> keeb:MX-10U-NoSwitch-ReversedStabilizers
- 7u1: renamed from 6.26u1; footprint MX_Only:MXOnly-6.25U-NoLED -> MX_Only:MXOnly-7U-ReversedStabilizers-NoLED
- C1: footprint Footprints:C_0805_2012Metric -> keeb:C_0805_2012Metric; moved to B.Cu
- D1, D10, D11, D12, D13, D14, D15, D16, D17, D18, D19, D2, D20, D21, D22, D23, D24, D25, D26, D27, D28, D29, D3, D30, D31, D32, D33, D34, D35, D36, D37, D38, D39, D4, D40, D41, D42, D43, D44, D45, D46, D47, D48, D49, D5, D50, D51, D52, D53, D54, D55, D56, D57, D58, D59, D6, D60, D61, D62, D63, D64, D65, D66, D67, D68, D69, D7, D70, D8, D9: footprint Footprints:D_SOD-123-Pretty -> keeb:D_SOD-123-Pretty; moved to B.Cu
- J1: footprint Footprints:JST-SR-4 -> keeb:JST-SR-4; moved to B.Cu
- JP1: footprint Footprints:ResetJumper -> keeb:ResetJumper; moved to B.Cu
- R1, R2, R3, R4, R5: footprint Footprints:R_0805_2012Metric -> keeb:R_0805_2012Metric; moved to B.Cu
- U1: footprint Package_QFP:TQFP-44_10x10mm_P0.8mm -> keeb:QFN_TQFP-44_Combined; moved to B.Cu
- Y1: value Resonator_Small -> Crystal_GND24_Small; footprint Footprints:Resonator_SMD_muRata_CSTxExxV-3Pin_3.0x1.1mm -> keeb:Crystal_SMD_3225-4Pin_3.2x2.5mm_HandSoldering; moved to B.Cu
- moved D70 323.9 mm to (325.1, 144.2), turned to 90 degrees
- moved JP1 323.6 mm to (291.0, 91.5), turned to 180 degrees
- moved D35 305.0 mm to (325.1, 87.0), turned to 90 degrees
- moved D33 300.6 mm to (287.0, 87.0), turned to 90 degrees
- moved 7u1 295.7 mm to (122.8, 139.2)
- moved D62 294.9 mm to (306.1, 125.1), turned to 90 degrees
- moved D61 290.0 mm to (263.2, 125.2), turned to 90 degrees
- moved D69 285.3 mm to (306.1, 144.2), turned to 90 degrees
- moved D67 274.1 mm to (258.4, 144.2), turned to 90 degrees
- moved D60 271.3 mm to (237.0, 125.2), turned to 90 degrees
- moved D66 264.0 mm to (210.8, 144.2), turned to 90 degrees
- moved D48 262.5 mm to (251.3, 106.1), turned to 90 degrees
- moved D47 260.5 mm to (220.3, 106.1), turned to 90 degrees
- moved D68 251.1 mm to (288.0, 139.7), turned to 90 degrees
- moved D18 250.0 mm to (325.1, 68.0), turned to 90 degrees
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Connections:
- MX55 pad 1: unconnected-(MX55-Pad1) -> COL14
- U1 pad 31: unconnected-(U1-Pad31) -> ROW2
- U1 pad 32: unconnected-(U1-Pad32) -> COL14
- U1 pad 36: unconnected-(U1-Pad36) -> COL11
- U1 pad 37: unconnected-(U1-Pad37) -> COL10
- U1 pad 38: unconnected-(U1-Pad38) -> COL9
- U1 pad 39: unconnected-(U1-Pad39) -> COL8
- U1 pad 40: unconnected-(U1-Pad40) -> COL7
- U1 pad 41: unconnected-(U1-Pad41) -> COL6
Routing:
- net ROW4: track 0.00 -> 333.6 mm
- net ROW0: track 0.00 -> 332.3 mm, vias 0 -> 2
- net ROW1: track 0.00 -> 323.9 mm, vias 0 -> 2
- net ROW3: track 0.00 -> 299.5 mm
- net ROW2: track 0.00 -> 289.1 mm
- net COL6: track 0.00 -> 260.9 mm
- net COL7: track 0.00 -> 221.1 mm
- net COL8: track 0.00 -> 202.8 mm
- net COL11: track 0.00 -> 190.5 mm
- net COL10: track 0.00 -> 184.5 mm
- net COL9: track 0.00 -> 184.2 mm
- net +5V: track 0.00 -> 149.4 mm, vias 0 -> 6
- net COL14: track 0.00 -> 133.8 mm
- net GND: track 0.00 -> 97.7 mm
- net COL0: track 0.00 -> 90.8 mm
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
Commit message: uh
Routing:
- net ROW4: track 333.6 -> 611.6 mm
- net ROW3: track 299.5 -> 556.9 mm, vias 0 -> 2
- net GND: track 97.7 -> 332.3 mm
- net COL0: track 90.8 -> 323.6 mm
- net LED: track 0.00 -> 232.6 mm
- net COL1: track 90.0 -> 290.4 mm
- net COL2: track 67.0 -> 247.4 mm
- net COL3: track 67.0 -> 227.5 mm
- net COL4: track 67.1 -> 207.5 mm
- net COL5: track 67.0 -> 187.5 mm
- net Net-(1.75u2-Pad2): track 9.53 -> 20.5 mm

Commit message: finish v1
Parts:
- added G***: LOGO, graphics:lg, F.Cu at (137.2, 138.7)
- added G***: LOGO, graphics:lg, B.Cu at (137.2, 138.7)
- 10u1: footprint keeb:MX-10U-NoSwitch-ReversedStabilizers -> keeb:MX-8U-NoSwitch
- moved D47 5.10 mm to (221.3, 101.1)
- moved D48 5.10 mm to (252.3, 101.1)
- turned 10u1 to 180 degrees
Connections:
- U1 pad 20: unconnected-(U1-Pad20) -> COL5
- U1 pad 21: unconnected-(U1-Pad21) -> COL4
- U1 pad 22: unconnected-(U1-Pad22) -> COL3
- U1 pad 25: unconnected-(U1-Pad25) -> COL2
- U1 pad 26: unconnected-(U1-Pad26) -> COL1
- U1 pad 27: unconnected-(U1-Pad27) -> COL0
- U1 pad 28: unconnected-(U1-Pad28) -> ROW3
- U1 pad 29: unconnected-(U1-Pad29) -> ROW4
- U1 pad 30: unconnected-(U1-Pad30) -> LED
Routing:
- net COL5: track 187.5 -> 281.3 mm
- net COL4: track 207.5 -> 297.1 mm
- net COL3: track 227.5 -> 314.0 mm
- net COL2: track 247.4 -> 324.3 mm
- net COL1: track 290.4 -> 365.3 mm
- net COL0: track 323.6 -> 397.3 mm
- net ROW3: track 556.9 -> 627.8 mm, vias 2 -> 0
- net ROW4: track 611.6 -> 681.1 mm
- net LED: track 232.6 -> 299.6 mm
- net GND: track 332.3 -> 399.2 mm, vias 0 -> 9
- net COL15: track 76.2 -> 90.9 mm, vias 2 -> 0
- net +5V: track 149.4 -> 142.3 mm
- net Net-(D47-Pad2): track 12.0 -> 7.45 mm
- net Net-(2.25u1-Pad2): track 12.2 -> 7.60 mm
- net ROW2: track 289.1 -> 292.6 mm
- added copper zone on B.Cu, net GND
- added copper zone on F.Cu, net GND
