File: KiCad/latte.kicad_pcb (KiCad board)
At the start: 2 copper layers, 347.8 x 94.7 mm, 163 parts, among them J1 Conn_01x04, U1 ATmega32U4-AU, Y1 Crystal_GND24_Small

Commit message: update README.md
Routing:
- net GND: vias 9 -> 10
Changed lines of the file:
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@@
       (effects (font (size 1 1) (thickness 0.15)) (justify mirror))
     )
-    (fp_text user "RESET" (at -0.02 -1.95) (layer "F.SilkS")
+    (fp_text user "RESET" (at -0.719 -2.074) (layer "F.SilkS")
       (effects (font (size 1 1) (thickness 0.15)))
     )
@@
   (segment (start 142.3 89.569359) (end 256.525 89.569359) (width 0.25) (layer "B.Cu") (net 21))
   (segment (start 268.994436 105.142822) (end 268.982178 105.142822) (width 0.25) (layer "B.Cu") (net 21))
-  (segment (start 257.680641 89.569359) (end 258.108665 89.569359) (width 0.25) (layer "B.Cu") (net 21))
   (segment (start 262.4 91.875) (end 260.094359 89.569359) (width 0.25) (layer "B.Cu") (net 21))
   (segment (start 262.4 103.903348) (end 262.4 91.875) (width 0.25) (layer "B.Cu") (net 21))
@@
   (via (at 256.65998 104.02002) (size 0.8) (drill 0.4) (layers "F.Cu" "B.Cu") (net 22))
   (via (at 270.9235 111.4735) (size 0.8) (drill 0.4) (layers "F.Cu" "B.Cu") (net 22))
+  (via (at 274.193 94.107) (size 0.8) (drill 0.4) (layers "F.Cu" "B.Cu") (free) (net 22))
   (via (at 210.82 147.193) (size 0.8) (drill 0.4) (layers "F.Cu" "B.Cu") (free) (net 22))
   (via (at 211.074 109.22) (size 0.8) (drill 0.4) (layers "F.Cu" "B.Cu") (free) (net 22))
@@
   (segment (start 269.449944 78.841945) (end 266.962087 81.329802) (width 0.381) (layer "B.Cu") (net 22))
   (segment (start 267.325545 95.412913) (end 270.125807 98.213175) (width 0.25) (layer "B.Cu") (net 23))
-  (segment (start 270.125807 98.213175) (end 270.113175 98.213175) (width 0.25) (layer "B.Cu") (net 23))
   (segment (start 266.887913 95.412913) (end 267.325545 95.412913) (width 0.25) (layer "B.Cu") (net 23))
   (segment (start 270.820465 69.625) (end 267.810425 69.625) (width 0.25) (layer "F.Cu") (net 24))
@@
   (segment (start 263.82548 89.85048) (end 263.82548 87.75048) (width 0.25) (layer "B.Cu") (net 100))
   (segment (start 263.82548 87.75048) (end 263.82548 86.56298) (width 0.25) (layer "B.Cu") (net 100))
-  (segment (start 268.428751 104.577136) (end 268.422864 104.577136) (width 0.25) (layer "B.Cu") (net 101))
   (segment (start 284.975 98.125) (end 283.275 98.125) (width 0.25) (layer "B.Cu") (net 104))
   (segment (start 281.95 96.8) (end 279.6 96.8) (width 0.25) (layer "B.Cu") (net 104))
@@
   (segment (start 280.654973 113.166463) (end 280.654973 111.005083) (width 0.25) (layer "B.Cu") (net 115))
   (segment (start 34.360705 109.501441) (end 34.908593 110.049329) (width 0.25) (layer "B.Cu") (net 115))
-  (segment (start 278.238031 115.583405) (end 278.238031 115.588969) (width 0.25) (layer "B.Cu") (net 115))
   (segment (start -2.7875 109.075) (end -2.3625 109.5) (width 0.25) (layer "B.Cu") (net 115))
   (segment (start 209.172837 104.744531) (end 258.155224 104.744531) (width 0.25) (layer "B.Cu") (net 115))
